Commit message: robot urdf

File: src/smart_robot/urdf/smart_robot.urdf.xacro (robot description, xacro)
@@ -1,48 +1,24 @@
 <?xml version="1.0"?>
-<robot xmlns:xacro="http://www.ros.org/wiki/xacro" name="smart_bot">
-    <!-- 定義一些常用的常數 -->
-    <xacro:property name="base_radius" value="0.15" /> <!-- 底盤半徑 -->
-    <xacro:property name="base_height" value="0.1" />  <!-- 底盤高度 -->
-    <xacro:property name="wheel_radius" value="0.05" /> <!-- 輪子半徑 -->
-    <xacro:property name="wheel_width" value="0.02" />  <!-- 輪子寬度 -->
-    <xacro:property name="caster_radius" value="0.025" /> <!-- 滾珠輪半徑 -->
-    <xacro:property name="laser_size" value="0.05" /> <!-- 雷射尺寸 -->
-    <!-- 慣性矩陣計算的宏 -->
-    <xacro:macro name="box_inertia" params="m w h d">
-        <inertial>
-            <mass value="${m}"/>
-            <inertia ixx="${m*(h*h+d*d)/12}" ixy="0" ixz="0" iyy="${m*(w*w+d*d)/12}" iyz="0" izz="${m*(w*w+h*h)/12}"/>
-        </inertial>
-    </xacro:macro>
+<robot xmlns:xacro="http://www.ros.org/wiki/xacro" name="smart_robot">
+    <!-- 常數定義 -->
+    <xacro:property name="PI" value="3.1415926535897931"/>
+    <xacro:property name="chassis_mass" value="1.0"/>
+    <xacro:property name="wheel_mass" value="0.1"/>
+    <xacro:property name="caster_mass" value="0.05"/>
+    <xacro:property name="chassis_radius" value="0.15"/>
+    <xacro:property name="chassis_height" value="0.1"/>
+    <xacro:property name="wheel_radius" value="0.05"/>
+    <xacro:property name="wheel_length" value="0.04"/>
+    <xacro:property name="wheel_separation" value="0.35"/> <!-- 兩個輪子之間的距離 -->
+    <!-- 慣性矩陣宏 -->
     <xacro:macro name="cylinder_inertia" params="m r h">
-        <inertial>
-            <mass value="${m}"/>
-            <inertia ixx="${m*(3*r*r+h*h)/12}" ixy="0" ixz="0" iyy="${m*(3*r*r+h*h)/12}" iyz="0" izz="${m*r*r/2}"/>
-        </inertial>
+        <inertia ixx="${m*(3*r*r+h*h)/12}" ixy="0" ixz="0" iyy="${m*(3*r*r+h*h)/12}" iyz="0" izz="${m*r*r/2}"/>
     </xacro:macro>
     <xacro:macro name="sphere_inertia" params="m r">
-        <inertial>
-            <mass value="${m}"/>
-            <inertia ixx="${2*m*r*r/5}" ixy="0" ixz="0" iyy="${2*m*r*r/5}" iyz="0" izz="${2*m*r*r/5}"/>
-        </inertial>
+        <inertia ixx="${2*m*r*r/5}" ixy="0" ixz="0" iyy="${2*m*r*r/5}" iyz="0" izz="${2*m*r*r/5}"/>
     </xacro:macro>
-    <!-- 1. 機器人主體 (底盤) -->
+    <!-- 機器人基礎 (通常是看不見的，用來穩定 TF tree) -->
     <link name="base_footprint"/>
-    <link name="base_link">
-        <visual>
-            <geometry>
-                <cylinder radius="${base_radius}" length="${base_height}"/>
-            </geometry>
-            <material name="blue">
-                <color rgba="0.2 0.6 1.0 1.0"/>
-            </material>
-        </visual>
-        <collision>
-            <geometry>
-                <cylinder radius="${base_radius}" length="${base_height}"/>
-            </geometry>
-        </collision>
-        <xacro:cylinder_inertia m="5.0" r="${base_radius}" h="${base_height}"/>
-    </link>
+    <!-- 車體 (chassis) -->
     <joint name="base_joint" type="fixed">
         <parent link="base_footprint"/>
@@ -50,117 +26,124 @@
         <origin xyz="0 0 ${wheel_radius}" rpy="0 0 0"/>
     </joint>
-    <!-- 2. 右輪 -->
-    <link name="right_wheel">
+    <link name="base_link">
         <visual>
-            <geometry>
-                <cylinder radius="${wheel_radius}" length="${wheel_width}"/>
-            </geometry>
-            <material name="black">
-                <color rgba="0.1 0.1 0.1 1.0"/>
-            </material>
+            <geometry><cylinder radius="${chassis_radius}" length="${chassis_height}"/></geometry>
+            <material name="blue"><color rgba="0.2 0.2 1.0 1.0"/></material>
         </visual>
         <collision>
-            <geometry>
-                <cylinder radius="${wheel_radius}" length="${wheel_width}"/>
-            </geometry>
+            <geometry><cylinder radius="${chassis_radius}" length="${chassis_height}"/></geometry>
         </collision>
-        <xacro:cylinder_inertia m="0.5" r="${wheel_radius}" h="${wheel_width}"/>
+        <inertial>
+            <mass value="${chassis_mass}"/>
+            <origin xyz="0 0 0"/>
+            <xacro:cylinder_inertia m="${chassis_mass}" r="${chassis_radius}" h="${chassis_height}"/>
+        </inertial>
     </link>
+    <!-- 右輪 -->
     <joint name="right_wheel_joint" type="continuous">
         <parent link="base_link"/>
-        <child link="right_wheel"/>
-        <origin xyz="0 -${base_radius} -${base_height/2 - wheel_radius}" rpy="-${pi/2} 0 0"/>
+        <child link="right_wheel_link"/>
+        <origin xyz="0 -${wheel_separation/2} 0" rpy="-${PI/2} 0 0"/>
         <axis xyz="0 0 1"/>
     </joint>
-    <!-- 3. 左輪 -->
-    <link name="left_wheel">
+    <link name="right_wheel_link">
         <visual>
-            <geometry>
-                <cylinder radius="${wheel_radius}" length="${wheel_width}"/>
-            </geometry>
+            <geometry><cylinder radius="${wheel_radius}" length="${wheel_length}"/></geometry>
+            <material name="black"><color rgba="0.1 0.1 0.1 1.0"/></material>
+        </visual>
+        <collision>
+            <geometry><cylinder radius="${wheel_radius}" length="${wheel_length}"/></geometry>
+        </collision>
+        <inertial>
+            <mass value="${wheel_mass}"/>
+            <xacro:cylinder_inertia m="${wheel_mass}" r="${wheel_radius}" h="${wheel_length}"/>
+        </inertial>
+    </link>
+    <!-- 左輪 -->
+    <joint name="left_wheel_joint" type="continuous">
+        <parent link="base_link"/>
+        <child link="left_wheel_link"/>
+        <origin xyz="0 ${wheel_separation/2} 0" rpy="${PI/2} 0 0"/>
+        <axis xyz="0 0 -1"/>
+    </joint>
+    <link name="left_wheel_link">
+        <visual>
+            <geometry><cylinder radius="${wheel_radius}" length="${wheel_length}"/></geometry>
             <material name="black"/>
         </visual>
         <collision>
-            <geometry>
-                <cylinder radius="${wheel_radius}" length="${wheel_width}"/>
-            </geometry>
+            <geometry><cylinder radius="${wheel_radius}" length="${wheel_length}"/></geometry>
         </collision>
-        <xacro:cylinder_inertia m="0.5" r="${wheel_radius}" h="${wheel_width}"/>
+        <inertial>
+            <mass value="${wheel_mass}"/>
+            <xacro:cylinder_inertia m="${wheel_mass}" r="${wheel_radius}" h="${wheel_length}"/>
+        </inertial>
     </link>
-    <joint name="left_wheel_joint" type="continuous">
+    <!-- 腳輪 (Caster Wheel) -->
+    <joint name="caster_wheel_joint" type="fixed">
         <parent link="base_link"/>
-        <child link="left_wheel"/>
-        <origin xyz="0 ${base_radius} -${base_height/2 - wheel_radius}" rpy="${pi/2} 0 0"/>
-        <axis xyz="0 0 -1"/>
+        <child link="caster_wheel_link"/>
+        <origin xyz="${chassis_radius*0.8} 0 -${wheel_radius*0.5}" rpy="0 0 0"/>
     </joint>
-    <!-- 4. 前方滾珠輪 -->
-    <link name="caster_wheel">
+    <link name="caster_wheel_link">
         <visual>
-            <geometry>
-                <sphere radius="${caster_radius}"/>
-            </geometry>
-            <material name="grey">
-                <color rgba="0.5 0.5 0.5 1.0"/>
-            </material>
+            <geometry><sphere radius="${wheel_radius*0.5}"/></geometry>
+            <material name="grey"><color rgba="0.5 0.5 0.5 1.0"/></material>
         </visual>
         <collision>
-            <geometry>
-                <sphere radius="${caster_radius}"/>
-            </geometry>
+            <geometry><sphere radius="${wheel_radius*0.5}"/></geometry>
         </collision>
-        <xacro:sphere_inertia m="0.3" r="${caster_radius}"/>
+        <inertial>
+            <mass value="${caster_mass}"/>
+            <xacro:sphere_inertia m="${caster_mass}" r="${wheel_radius*0.5}"/>
+        </inertial>
     </link>
-    <joint name="caster_wheel_joint" type="fixed">
-        <parent link="base_link"/>
-        <child link="caster_wheel"/>
-        <origin xyz="${base_radius*0.8} 0 -${base_height/2 - caster_radius}" rpy="0 0 0"/>
-    </joint>
-    <!-- 5. 雷射掃描儀 (LIDAR) -->
-    <link name="laser_link">
-        <visual>
-            <geometry>
-                <cylinder radius="${laser_size}" length="${laser_size}"/>
-            </geometry>
-            <material name="red">
-                <color rgba="1.0 0.0 0.0 1.0"/>
-            </material>
-        </visual>
-        <collision>
-            <geometry>
-                <cylinder radius="${laser_size}" length="${laser_size}"/>
-            </geometry>
-        </collision>
-        <xacro:cylinder_inertia m="0.1" r="${laser_size}" h="${laser_size}"/>
-    </link>
+    <!-- 雷射掃描儀 (Lidar) -->
     <joint name="laser_joint" type="fixed">
         <parent link="base_link"/>
         <child link="laser_link"/>
-        <origin xyz="0 0 ${base_height/2 + laser_size/2}" rpy="0 0 0"/>
+        <!-- *** 關鍵點：將雷射放在車體頂部，避免掃描到自己或地面 *** -->
+        <origin xyz="0 0 ${chassis_height/2 + 0.02}" rpy="0 0 0"/>
     </joint>
-    <!-- Gazebo 插件 -->
-    <!-- 1. 差速驅動插件 (讓輪子動起來) -->
+    <link name="laser_link">
+        <visual>
+            <geometry><cylinder radius="0.05" length="0.04"/></geometry>
+            <material name="red"><color rgba="1.0 0.0 0.0 1.0"/></material>
+        </visual>
+        <collision>
+            <geometry><cylinder radius="0.05" length="0.04"/></geometry>
+        </collision>
+        <inertial>
+            <mass value="0.1"/>
+            <xacro:cylinder_inertia m="0.1" r="0.05" h="0.04"/>
+        </inertial>
+    </link>
+    <!-- ################# GAZEBO PLUGINS ################# -->
+    <!-- 差速驅動插件 -->
     <gazebo>
-        <plugin name="differential_drive_controller" filename="libgazebo_ros_diff_drive.so">
+        <plugin name="diff_drive_controller" filename="libgazebo_ros_diff_drive.so">
             <alwaysOn>true</alwaysOn>
-            <updateRate>100</updateRate>
-            <leftJoint>left_wheel_joint</leftJoint>
+            <updateRate>50</updateRate>
+            <leftJoint>left_wheel_joint</leftJoint>   <!-- *** 關鍵點：指定左右輪關節 *** -->
             <rightJoint>right_wheel_joint</rightJoint>
-            <wheelSeparation>${base_radius*2}</wheelSeparation>
+            <wheelSeparation>${wheel_separation}</wheelSeparation>
             <wheelDiameter>${wheel_radius*2}</wheelDiameter>
-            <torque>20</torque>
-            <!-- 這個插件會訂閱 /cmd_vel 主題 -->
-            <commandTopic>cmd_vel</commandTopic>
-            <!-- 這個插件會發布 odom 主題 -->
-            <odometryTopic>odom</odometryTopic>
+            <wheelTorque>20</wheelTorque>
+            <wheelAcceleration>1.8</wheelAcceleration>
+            <commandTopic>cmd_vel</commandTopic>   <!-- *** 關鍵點：指定訂閱的話題 *** -->
+            <odometryTopic>odom</odometryTopic>     <!-- *** 關鍵點：指定發布里程計的話題 *** -->
             <odometryFrame>odom</odometryFrame>
             <robotBaseFrame>base_footprint</robotBaseFrame>
+            <publishWheelTF>false</publishWheelTF>
+            <publishOdomTF>true</publishOdomTF>
+            <publishWheelJointState>true</publishWheelJointState>
         </plugin>
     </gazebo>
-    <!-- 2. 雷射掃描儀插件 -->
+    <!-- 雷射插件 -->
     <gazebo reference="laser_link">
-        <sensor type="ray" name="laser_sensor">
+        <sensor type="ray" name="head_hokuyo_sensor">
             <pose>0 0 0 0 0 0</pose>
-            <visualize>true</visualize>
-            <update_rate>10</update_rate>
+            <visualize>false</visualize>
+            <update_rate>20</update_rate>
             <ray>
                 <scan>
@@ -168,16 +151,20 @@
                         <samples>360</samples>
                         <resolution>1</resolution>
-                        <min_angle>-3.14159</min_angle>
-                        <max_angle>3.14159</max_angle>
+                        <min_angle>-${PI}</min_angle>
+                        <max_angle>${PI}</max_angle>
                     </horizontal>
                 </scan>
                 <range>
-                    <min>0.1</min>
-                    <max>12.0</max>
+                    <min>0.10</min>
+                    <max>10.0</max>
                     <resolution>0.01</resolution>
                 </range>
+                <noise>
+                    <type>gaussian</type>
+                    <mean>0.0</mean>
+                    <stddev>0.01</stddev>
+                </noise>
             </ray>
-            <plugin name="gazebo_ros_laser" filename="libgazebo_ros_laser.so">
-                <!-- 這個插件會發布 /scan 主題 -->
+            <plugin name="gazebo_ros_head_hokuyo_controller" filename="libgazebo_ros_laser.so">
                 <topicName>/scan</topicName>
                 <frameName>laser_link</frameName>

Commit message: decline wheel

File: src/smart_robot/urdf/smart_robot.urdf.xacro (robot description, xacro)
@@ -10,5 +10,5 @@
     <xacro:property name="wheel_radius" value="0.05"/>
     <xacro:property name="wheel_length" value="0.04"/>
-    <xacro:property name="wheel_separation" value="0.35"/> <!-- 兩個輪子之間的距離 -->
+    <xacro:property name="wheel_separation" value="0.35"/>
     <!-- 慣性矩陣宏 -->
     <xacro:macro name="cylinder_inertia" params="m r h">
@@ -84,5 +84,5 @@
         <parent link="base_link"/>
         <child link="caster_wheel_link"/>
-        <origin xyz="${chassis_radius*0.8} 0 -${wheel_radius*0.5}" rpy="0 0 0"/>
+        <origin xyz="${chassis_radius*0.8} 0 0" rpy="0 0 0"/>
     </joint>
     <link name="caster_wheel_link">

Commit message: add friction

File: src/smart_robot/urdf/smart_robot.urdf.xacro (robot description, xacro)
@@ -59,4 +59,11 @@
             <xacro:cylinder_inertia m="${wheel_mass}" r="${wheel_radius}" h="${wheel_length}"/>
         </inertial>
+        <gazebo reference="right_wheel_link">
+            <mu1>1.0</mu1>
+            <mu2>1.0</mu2>
+            <kp>1000000.0</kp>
+            <kd>100.0</kd>
+            <material>Gazebo/Grey</material>
+        </gazebo>
     </link>
     <!-- 左輪 -->
@@ -79,4 +86,11 @@
             <xacro:cylinder_inertia m="${wheel_mass}" r="${wheel_radius}" h="${wheel_length}"/>
         </inertial>
+        <gazebo reference="left_wheel_link">
+            <mu1>1.0</mu1>
+            <mu2>1.0</mu2>
+            <kp>1000000.0</kp>
+            <kd>100.0</kd>
+            <material>Gazebo/Grey</material>
+        </gazebo>
     </link>
     <!-- 腳輪 (Caster Wheel) -->
@@ -98,4 +112,11 @@
             <xacro:sphere_inertia m="${caster_mass}" r="${wheel_radius*0.5}"/>
         </inertial>
+        <gazebo reference="caster_wheel_link">
+            <mu1>0.1</mu1>
+            <mu2>0.1</mu2>
+            <kp>1000000.0</kp>
+            <kd>100.0</kd>
+            <material>Gazebo/Grey</material>
+        </gazebo>
     </link>
     <!-- 雷射掃描儀 (Lidar) -->

Commit message: elevate chassis

File: src/smart_robot/urdf/smart_robot.urdf.xacro (robot description, xacro)
@@ -24,5 +24,5 @@
         <parent link="base_footprint"/>
         <child link="base_link"/>
-        <origin xyz="0 0 ${wheel_radius}" rpy="0 0 0"/>
+        <origin xyz="0 0 ${wheel_radius + 0.02}" rpy="0 0 0"/>
     </joint>
     <link name="base_link">

Commit message: elevate chassis

File: src/smart_robot/urdf/smart_robot.urdf.xacro (robot description, xacro)
@@ -24,5 +24,5 @@
         <parent link="base_footprint"/>
         <child link="base_link"/>
-        <origin xyz="0 0 ${wheel_radius + 0.02}" rpy="0 0 0"/>
+        <origin xyz="0 0 ${wheel_radius + 0.5}" rpy="0 0 0"/>
     </joint>
     <link name="base_link">

Commit message: elevate chassis

File: src/smart_robot/urdf/smart_robot.urdf.xacro (robot description, xacro)
@@ -24,5 +24,5 @@
         <parent link="base_footprint"/>
         <child link="base_link"/>
-        <origin xyz="0 0 ${wheel_radius + 0.5}" rpy="0 0 0"/>
+        <origin xyz="0 0 ${chassis_height/2 + 0.01}" rpy="0 0 0"/>
     </joint>
     <link name="base_link">
@@ -44,5 +44,5 @@
         <parent link="base_link"/>
         <child link="right_wheel_link"/>
-        <origin xyz="0 -${wheel_separation/2} 0" rpy="-${PI/2} 0 0"/>
+        <origin xyz="0 -${wheel_separation/2} -0.01" rpy="-${PI/2} 0 0"/>
         <axis xyz="0 0 1"/>
     </joint>
@@ -67,9 +67,9 @@
         </gazebo>
     </link>
-    <!-- 左輪 -->
+     <!-- 左輪 -->
     <joint name="left_wheel_joint" type="continuous">
         <parent link="base_link"/>
         <child link="left_wheel_link"/>
-        <origin xyz="0 ${wheel_separation/2} 0" rpy="${PI/2} 0 0"/>
+        <origin xyz="0 ${wheel_separation/2} -0.01" rpy="${PI/2} 0 0"/>
         <axis xyz="0 0 -1"/>
     </joint>
@@ -98,5 +98,5 @@
         <parent link="base_link"/>
         <child link="caster_wheel_link"/>
-        <origin xyz="${chassis_radius*0.8} 0 0" rpy="0 0 0"/>
+        <origin xyz="${chassis_radius*0.8} 0 -0.035" rpy="0 0 0"/>
     </joint>
     <link name="caster_wheel_link">

Commit message: lazer decline & add wheel

File: src/smart_robot/urdf/smart_robot.urdf.xacro (robot description, xacro)
@@ -94,5 +94,5 @@
         </gazebo>
     </link>
-    <!-- 腳輪 (Caster Wheel) -->
+    <!-- 前腳輪 (Caster Wheel) -->
     <joint name="caster_wheel_joint" type="fixed">
         <parent link="base_link"/>
@@ -120,9 +120,35 @@
         </gazebo>
     </link>
+    <!-- 後腳輪 (Caster Wheel) -->
+    <joint name="caster_wheel_rear_joint" type="fixed">
+        <parent link="base_link"/>
+        <child link="caster_wheel_rear_link"/>
+        <origin xyz="-${chassis_radius*0.8} 0 -0.035" rpy="0 0 0"/>
+    </joint>
+    <link name="caster_wheel_link">
+        <visual>
+            <geometry><sphere radius="${wheel_radius*0.5}"/></geometry>
+            <material name="grey"><color rgba="0.5 0.5 0.5 1.0"/></material>
+        </visual>
+        <collision>
+            <geometry><sphere radius="${wheel_radius*0.5}"/></geometry>
+        </collision>
+        <inertial>
+            <mass value="${caster_mass}"/>
+            <xacro:sphere_inertia m="${caster_mass}" r="${wheel_radius*0.5}"/>
+        </inertial>
+        <gazebo reference="caster_wheel_link">
+            <mu1>0.1</mu1>
+            <mu2>0.1</mu2>
+            <kp>1000000.0</kp>
+            <kd>100.0</kd>
+            <material>Gazebo/Grey</material>
+        </gazebo>
+    </link>
     <!-- 雷射掃描儀 (Lidar) -->
     <joint name="laser_joint" type="fixed">
         <parent link="base_link"/>
         <child link="laser_link"/>
-        <origin xyz="0 0 ${chassis_height/2 + 0.02}" rpy="0 0 0"/>
+        <origin xyz="${chassis_radius} 0 -0.01" rpy="0 0 0"/>
     </joint>
     <link name="laser_link">

Commit message: wheel name bug

File: src/smart_robot/urdf/smart_robot.urdf.xacro (robot description, xacro)
@@ -94,11 +94,11 @@
         </gazebo>
     </link>
-    <!-- 前腳輪 (Caster Wheel) -->
-    <joint name="caster_wheel_joint" type="fixed">
-        <parent link="base_link"/>
-        <child link="caster_wheel_link"/>
+    <!-- 前腳輪 (Front Caster Wheel) -->
+    <joint name="caster_wheel_front_joint" type="fixed">
+        <parent link="base_link"/>
+        <child link="caster_wheel_front_link"/>
         <origin xyz="${chassis_radius*0.8} 0 -0.035" rpy="0 0 0"/>
     </joint>
-    <link name="caster_wheel_link">
+    <link name="caster_wheel_front_link">
         <visual>
             <geometry><sphere radius="${wheel_radius*0.5}"/></geometry>
@@ -112,13 +112,11 @@
             <xacro:sphere_inertia m="${caster_mass}" r="${wheel_radius*0.5}"/>
         </inertial>
-        <gazebo reference="caster_wheel_link">
+        <gazebo reference="caster_wheel_front_link">
             <mu1>0.1</mu1>
             <mu2>0.1</mu2>
-            <kp>1000000.0</kp>
-            <kd>100.0</kd>
-            <material>Gazebo/Grey</material>
-        </gazebo>
-    </link>
-    <!-- 後腳輪 (Caster Wheel) -->
+            <material>Gazebo/Grey</material>
+        </gazebo>
+    </link>
+    <!-- 後腳輪 (Rear Caster Wheel) -->
     <joint name="caster_wheel_rear_joint" type="fixed">
         <parent link="base_link"/>
@@ -126,8 +124,8 @@
         <origin xyz="-${chassis_radius*0.8} 0 -0.035" rpy="0 0 0"/>
     </joint>
-    <link name="caster_wheel_link">
-        <visual>
-            <geometry><sphere radius="${wheel_radius*0.5}"/></geometry>
-            <material name="grey"><color rgba="0.5 0.5 0.5 1.0"/></material>
+    <link name="caster_wheel_rear_link">
+        <visual>
+            <geometry><sphere radius="${wheel_radius*0.5}"/></geometry>
+            <material name="grey"/>
         </visual>
         <collision>
@@ -138,9 +136,7 @@
             <xacro:sphere_inertia m="${caster_mass}" r="${wheel_radius*0.5}"/>
         </inertial>
-        <gazebo reference="caster_wheel_link">
+        <gazebo reference="caster_wheel_rear_link">
             <mu1>0.1</mu1>
             <mu2>0.1</mu2>
-            <kp>1000000.0</kp>
-            <kd>100.0</kd>
             <material>Gazebo/Grey</material>
         </gazebo>

Commit message: fix laser bug

File: src/smart_robot/urdf/smart_robot.urdf.xacro (robot description, xacro)
@@ -146,5 +146,5 @@
         <parent link="base_link"/>
         <child link="laser_link"/>
-        <origin xyz="${chassis_radius} 0 -0.01" rpy="0 0 0"/>
+        <origin xyz="0 0 -0.01" rpy="0 0 0"/>
     </joint>
     <link name="laser_link">
@@ -154,8 +154,8 @@
         </visual>
         <collision>
-            <geometry><cylinder radius="0.05" length="0.04"/></geometry>
-        </collision>
-        <inertial>
-            <mass value="0.1"/>
+            <geometry><cylinder radius="0.001" length="0.001"/></geometry>
+        </collision>
+        <inertial>
+            <mass value="0.001"/>
             <xacro:cylinder_inertia m="0.1" r="0.05" h="0.04"/>
         </inertial>

Commit message: fix laser bug

File: src/smart_robot/urdf/smart_robot.urdf.xacro (robot description, xacro)
@@ -146,5 +146,5 @@
         <parent link="base_link"/>
         <child link="laser_link"/>
-        <origin xyz="0 0 -0.01" rpy="0 0 0"/>
+        <origin xyz="${chassis_radius} 0 0.04" rpy="0 0 0"/>
     </joint>
     <link name="laser_link">
@@ -154,8 +154,8 @@
         </visual>
         <collision>
-            <geometry><cylinder radius="0.001" length="0.001"/></geometry>
-        </collision>
-        <inertial>
-            <mass value="0.001"/>
+            <geometry><cylinder radius="0.05" length="0.04"/></geometry>
+        </collision>
+        <inertial>
+            <mass value="0.1"/>
             <xacro:cylinder_inertia m="0.1" r="0.05" h="0.04"/>
         </inertial>
@@ -192,8 +192,8 @@
                 <scan>
                     <horizontal>
-                        <samples>360</samples>
+                        <samples>120</samples>
                         <resolution>1</resolution>
-                        <min_angle>-${PI}</min_angle>
-                        <max_angle>${PI}</max_angle>
+                        <min_angle>-${2*PI/3}</min_angle>
+                        <max_angle>${2*PI/3}</max_angle>
                     </horizontal>
                 </scan>
