Commit message: fix urdf

File: src/smart_robot/urdf/smart_robot.urdf.xacro (robot description, xacro)
@@ -23,25 +23,49 @@
         <inertial><mass value="${chassis_mass}"/><origin xyz="0 0 0"/><xacro:solid_cylinder_inertia m="${chassis_mass}" r="${chassis_radius}" h="${chassis_height}"/></inertial>
     </link>
+    <!-- RIGHT WHEEL -->
     <joint name="right_wheel_joint" type="continuous">
         <parent link="base_link"/>
         <child link="right_wheel_link"/>
-        <origin xyz="0 -${wheel_separation/2} -0.01" rpy="-${PI/2} 0 0"/>
-        <axis xyz="0 0 1"/>
+        <origin xyz="0 -${wheel_separation/2} -0.01" rpy="0 0 0"/>
+        <axis xyz="0 1 0"/> <!-- 旋轉軸沿著 Y 軸 -->
     </joint>
     <link name="right_wheel_link">
-        <visual><geometry><cylinder radius="${wheel_radius}" length="${wheel_length}"/></geometry><material name="black"><color rgba="0.1 0.1 0.1 1.0"/></material></visual>
-        <collision><geometry><cylinder radius="${wheel_radius}" length="${wheel_length}"/></geometry></collision>
-        <inertial><mass value="${wheel_mass}"/><xacro:wheel_inertia m="${wheel_mass}" r="${wheel_radius}" h="${wheel_length}"/></inertial>
+        <visual>
+            <origin xyz="0 0 0" rpy="${PI/2} 0 0"/>
+            <geometry><cylinder radius="${wheel_radius}" length="${wheel_length}"/></geometry>
+            <material name="black"><color rgba="0.1 0.1 0.1 1.0"/></material>
+        </visual>
+        <collision>
+            <origin xyz="0 0 0" rpy="${PI/2} 0 0"/>
+            <geometry><cylinder radius="${wheel_radius}" length="${wheel_length}"/></geometry>
+        </collision>
+        <inertial>
+            <mass value="${wheel_mass}"/>
+            <origin xyz="0 0 0" rpy="${PI/2} 0 0"/>
+            <xacro:wheel_inertia m="${wheel_mass}" r="${wheel_radius}" h="${wheel_length}"/>
+        </inertial>
     </link>
+    <!-- LEFT WHEEL -->
     <joint name="left_wheel_joint" type="continuous">
         <parent link="base_link"/>
         <child link="left_wheel_link"/>
-        <origin xyz="0 ${wheel_separation/2} -0.01" rpy="${PI/2} 0 0"/>
-        <axis xyz="0 0 1"/>
+        <origin xyz="0 ${wheel_separation/2} -0.01" rpy="0 0 0"/>
+        <axis xyz="0 -1 0"/>
     </joint>
     <link name="left_wheel_link">
-        <visual><geometry><cylinder radius="${wheel_radius}" length="${wheel_length}"/></geometry><material name="black"/></visual>
-        <collision><geometry><cylinder radius="${wheel_radius}" length="${wheel_length}"/></geometry></collision>
-        <inertial><mass value="${wheel_mass}"/><xacro:wheel_inertia m="${wheel_mass}" r="${wheel_radius}" h="${wheel_length}"/></inertial>
+        <visual>
+            <origin xyz="0 0 0" rpy="${PI/2} 0 0"/>
+            <geometry><cylinder radius="${wheel_radius}" length="${wheel_length}"/></geometry>
+            <material name="black"/>
+        </visual>
+        <collision>
+            <origin xyz="0 0 0" rpy="${PI/2} 0 0"/>
+            <geometry><cylinder radius="${wheel_radius}" length="${wheel_length}"/></geometry>
+        </collision>
+        <inertial>
+            <mass value="${wheel_mass}"/>
+            <origin xyz="0 0 0" rpy="${PI/2} 0 0"/>
+            <xacro:wheel_inertia m="${wheel_mass}" r="${wheel_radius}" h="${wheel_length}"/>
+        </inertial>
     </link>
     <joint name="caster_wheel_front_joint" type="fixed"><parent link="base_link"/><child link="caster_wheel_front_link"/><origin xyz="${chassis_radius*0.8} 0 -0.035" rpy="0 0 0"/></joint>

Commit message: fix robot

File: src/smart_robot/urdf/smart_robot.urdf.xacro (robot description, xacro)
@@ -17,5 +17,9 @@
     <!-- ================== ROBOT LINKS AND JOINTS ================== -->
     <link name="base_footprint"/>
-    <joint name="base_joint" type="fixed"><parent link="base_footprint"/><child link="base_link"/><origin xyz="0 0 ${chassis_height/2 + 0.01}" rpy="0 0 0"/></joint>
+    <joint name="base_joint" type="fixed">
+        <parent link="base_footprint"/>
+        <child link="base_link"/>
+        <origin xyz="0 0 ${chassis_height/2 + 0.01}" rpy="0 0 -${PI/2}"/>
+    </joint>
     <link name="base_link">
         <visual><geometry><cylinder radius="${chassis_radius}" length="${chassis_height}"/></geometry><material name="blue"><color rgba="0.2 0.2 1.0 1.0"/></material></visual>
@@ -28,5 +32,5 @@
         <child link="right_wheel_link"/>
         <origin xyz="0 -${wheel_separation/2} -0.01" rpy="0 0 0"/>
-        <axis xyz="0 1 0"/> <!-- 旋轉軸沿著 Y 軸 -->
+        <axis xyz="0 1 0"/>
     </joint>
     <link name="right_wheel_link">

Commit message: fix robot

File: src/smart_robot/urdf/smart_robot.urdf.xacro (robot description, xacro)
@@ -13,23 +13,39 @@
     <!-- ================== INERTIA MACROS ================== -->
     <xacro:macro name="solid_cylinder_inertia" params="m r h"><inertia ixx="${m*(3*r*r+h*h)/12}" ixy="0" ixz="0" iyy="${m*(3*r*r+h*h)/12}" iyz="0" izz="${m*r*r/2}"/></xacro:macro>
-    <xacro:macro name="wheel_inertia" params="m r h"><inertia ixx="${m*(3*r*r+h*h)/12}" ixy="0" ixz="0" iyy="${m*r*r/2}" iyz="0" izz="${m*(3*r*r+h*h)/12}"/></xacro:macro>
     <xacro:macro name="sphere_inertia" params="m r"><inertia ixx="${2*m*r*r/5}" ixy="0" ixz="0" iyy="${2*m*r*r/5}" iyz="0" izz="${2*m*r*r/5}"/></xacro:macro>
+    <xacro:macro name="wheel_inertia" params="m r h">
+      <inertia ixx="${(m/12.0)*(3*r*r + h*h)}" ixy="0.0" ixz="0.0"
+               iyy="${(m/2.0)*(r*r)}" iyz="0.0"
+               izz="${(m/12.0)*(3*r*r + h*h)}"/>
+    </xacro:macro>
     <!-- ================== ROBOT LINKS AND JOINTS ================== -->
+    <!-- Base Footprint: The 2D projection on the ground -->
     <link name="base_footprint"/>
     <joint name="base_joint" type="fixed">
         <parent link="base_footprint"/>
         <child link="base_link"/>
-        <origin xyz="0 0 ${chassis_height/2 + 0.01}" rpy="0 0 -${PI/2}"/>
+        <origin xyz="0 0 ${wheel_radius}" rpy="0 0 0"/>
     </joint>
     <link name="base_link">
-        <visual><geometry><cylinder radius="${chassis_radius}" length="${chassis_height}"/></geometry><material name="blue"><color rgba="0.2 0.2 1.0 1.0"/></material></visual>
-        <collision><geometry><cylinder radius="${chassis_radius}" length="${chassis_height}"/></geometry></collision>
-        <inertial><mass value="${chassis_mass}"/><origin xyz="0 0 0"/><xacro:solid_cylinder_inertia m="${chassis_mass}" r="${chassis_radius}" h="${chassis_height}"/></inertial>
+        <visual>
+            <geometry><cylinder radius="${chassis_radius}" length="${chassis_height}"/></geometry>
+            <origin xyz="0 0 0" rpy="0 0 0" />
+            <material name="blue"><color rgba="0.2 0.2 1.0 1.0"/></material>
+        </visual>
+        <collision>
+            <geometry><cylinder radius="${chassis_radius}" length="${chassis_height}"/></geometry>
+            <origin xyz="0 0 0" rpy="0 0 0" />
+        </collision>
+        <inertial>
+            <mass value="${chassis_mass}"/>
+            <origin xyz="0 0 0"/>
+            <xacro:solid_cylinder_inertia m="${chassis_mass}" r="${chassis_radius}" h="${chassis_height}"/>
+        </inertial>
     </link>
-    <!-- RIGHT WHEEL -->
+    <!-- RIGHT WHEEL: Placed on the -Y axis -->
     <joint name="right_wheel_joint" type="continuous">
         <parent link="base_link"/>
         <child link="right_wheel_link"/>
-        <origin xyz="0 -${wheel_separation/2} -0.01" rpy="0 0 0"/>
+        <origin xyz="0 -${wheel_separation/2} 0" rpy="0 0 0"/>
         <axis xyz="0 1 0"/>
     </joint>
@@ -50,10 +66,10 @@
         </inertial>
     </link>
-    <!-- LEFT WHEEL -->
+    <!-- LEFT WHEEL: Placed on the +Y axis -->
     <joint name="left_wheel_joint" type="continuous">
         <parent link="base_link"/>
         <child link="left_wheel_link"/>
-        <origin xyz="0 ${wheel_separation/2} -0.01" rpy="0 0 0"/>
-        <axis xyz="0 -1 0"/>
+        <origin xyz="0 ${wheel_separation/2} 0" rpy="0 0 0"/>
+        <axis xyz="0 1 0"/>
     </joint>
     <link name="left_wheel_link">
@@ -73,5 +89,10 @@
         </inertial>
     </link>
-    <joint name="caster_wheel_front_joint" type="fixed"><parent link="base_link"/><child link="caster_wheel_front_link"/><origin xyz="${chassis_radius*0.8} 0 -0.035" rpy="0 0 0"/></joint>
+    <!-- Caster Wheels -->
+    <joint name="caster_wheel_front_joint" type="fixed">
+        <parent link="base_link"/>
+        <child link="caster_wheel_front_link"/>
+        <origin xyz="${chassis_radius*0.8} 0 -${wheel_radius*0.5}" rpy="0 0 0"/>
+    </joint>
     <link name="caster_wheel_front_link">
         <visual><geometry><sphere radius="${wheel_radius*0.5}"/></geometry><material name="grey"><color rgba="0.5 0.5 0.5 1.0"/></material></visual>
@@ -79,5 +100,9 @@
         <inertial><mass value="${caster_mass}"/><xacro:sphere_inertia m="${caster_mass}" r="${wheel_radius*0.5}"/></inertial>
     </link>
-    <joint name="caster_wheel_rear_joint" type="fixed"><parent link="base_link"/><child link="caster_wheel_rear_link"/><origin xyz="-${chassis_radius*0.8} 0 -0.035" rpy="0 0 0"/></joint>
+    <joint name="caster_wheel_rear_joint" type="fixed">
+        <parent link="base_link"/>
+        <child link="caster_wheel_rear_link"/>
+        <origin xyz="-${chassis_radius*0.8} 0 -${wheel_radius*0.5}" rpy="0 0 0"/>
+    </joint>
     <link name="caster_wheel_rear_link">
         <visual><geometry><sphere radius="${wheel_radius*0.5}"/></geometry><material name="grey"/></visual>
@@ -85,5 +110,10 @@
         <inertial><mass value="${caster_mass}"/><xacro:sphere_inertia m="${caster_mass}" r="${wheel_radius*0.5}"/></inertial>
     </link>
-    <joint name="laser_joint" type="fixed"><parent link="base_link"/><child link="laser_link"/><origin xyz="0 0 0.06" rpy="0 0 0"/></joint>
+    <!-- Laser Scanner -->
+    <joint name="laser_joint" type="fixed">
+        <parent link="base_link"/>
+        <child link="laser_link"/>
+        <origin xyz="${chassis_radius*0.9} 0 ${chassis_height/2}" rpy="0 0 0"/>
+    </joint>
     <link name="laser_link">
         <visual><geometry><cylinder radius="0.05" length="0.04"/></geometry><material name="red"><color rgba="1.0 0.0 0.0 1.0"/></material></visual>
@@ -108,8 +138,40 @@
             <publishOdomTF>true</publishOdomTF>
             <odometrySource>world</odometrySource>
+            <!-- These are optional but good to have -->
+            <publishWheelTF>false</publishWheelTF>
+            <publishWheelJointState>true</publishWheelJointState>
+            <legacyMode>false</legacyMode>
         </plugin>
     </gazebo>
     <gazebo reference="laser_link">
-        <sensor type="ray" name="hokuyo_sensor"><pose>0 0 0 0 0 0</pose><visualize>true</visualize><update_rate>20</update_rate><ray><scan><horizontal><samples>360</samples><resolution>1</resolution><min_angle>-${PI}</min_angle><max_angle>${PI}</max_angle></horizontal></scan><range><min>0.10</min><max>10.0</max><resolution>0.01</resolution></range><noise><type>gaussian</type><mean>0.0</mean><stddev>0.01</stddev></noise></ray><plugin name="gazebo_ros_head_hokuyo_controller" filename="libgazebo_ros_laser.so"><topicName>/scan</topicName><frameName>laser_link</frameName></plugin></sensor>
+        <sensor type="ray" name="hokuyo_sensor">
+            <pose>0 0 0 0 0 0</pose>
+            <visualize>false</visualize>
+            <update_rate>20</update_rate>
+            <ray>
+                <scan>
+                    <horizontal>
+                        <samples>360</samples>
+                        <resolution>1</resolution>
+                        <min_angle>-${PI}</min_angle>
+                        <max_angle>${PI}</max_angle>
+                    </horizontal>
+                </scan>
+                <range>
+                    <min>0.10</min>
+                    <max>10.0</max>
+                    <resolution>0.01</resolution>
+                </range>
+                <noise>
+                    <type>gaussian</type>
+                    <mean>0.0</mean>
+                    <stddev>0.01</stddev>
+                </noise>
+            </ray>
+            <plugin name="gazebo_ros_head_hokuyo_controller" filename="libgazebo_ros_laser.so">
+                <topicName>/scan</topicName>
+                <frameName>laser_link</frameName>
+            </plugin>
+        </sensor>
     </gazebo>
 </robot>

Commit message: fix robot

File: src/smart_robot/urdf/smart_robot.urdf.xacro (robot description, xacro)
@@ -65,4 +65,11 @@
             <xacro:wheel_inertia m="${wheel_mass}" r="${wheel_radius}" h="${wheel_length}"/>
         </inertial>
+        <gazebo reference="right_wheel_link">
+            <mu1>1.0</mu1>
+            <mu2>1.0</mu2>
+            <kp>1000000.0</kp>
+            <kd>100.0</kd>
+            <material>Gazebo/Black</material>
+        </gazebo>
     </link>
     <!-- LEFT WHEEL: Placed on the +Y axis -->
@@ -88,4 +95,11 @@
             <xacro:wheel_inertia m="${wheel_mass}" r="${wheel_radius}" h="${wheel_length}"/>
         </inertial>
+        <gazebo reference="right_wheel_link">
+            <mu1>1.0</mu1>
+            <mu2>1.0</mu2>
+            <kp>1000000.0</kp>
+            <kd>100.0</kd>
+            <material>Gazebo/Black</material>
+        </gazebo>
     </link>
     <!-- Caster Wheels -->
@@ -99,4 +113,11 @@
         <collision><geometry><sphere radius="${wheel_radius*0.5}"/></geometry></collision>
         <inertial><mass value="${caster_mass}"/><xacro:sphere_inertia m="${caster_mass}" r="${wheel_radius*0.5}"/></inertial>
+        <gazebo reference="caster_wheel_front_link">
+            <mu1>0.05</mu1>
+            <mu2>0.05</mu2>
+            <kp>1000000.0</kp>
+            <kd>100.0</kd>
+            <material>Gazebo/Grey</material>
+        </gazebo>
     </link>
     <joint name="caster_wheel_rear_joint" type="fixed">
@@ -138,4 +159,6 @@
             <publishOdomTF>true</publishOdomTF>
             <odometrySource>world</odometrySource>
+            <leftJointPID>10.0 0.0 0.0</leftJointPID>
+            <rightJointPID>10.0 0.0 0.0</rightJointPID>
             <!-- These are optional but good to have -->
             <publishWheelTF>false</publishWheelTF>

Commit message: add damping

File: src/smart_robot/urdf/smart_robot.urdf.xacro (robot description, xacro)
@@ -49,4 +49,5 @@
         <origin xyz="0 -${wheel_separation/2} 0" rpy="0 0 0"/>
         <axis xyz="0 1 0"/>
+        <dynamics damping="0.1"/>
     </joint>
     <link name="right_wheel_link">
@@ -79,4 +80,5 @@
         <origin xyz="0 ${wheel_separation/2} 0" rpy="0 0 0"/>
         <axis xyz="0 1 0"/>
+        <dynamics damping="0.1"/>
     </joint>
     <link name="left_wheel_link">

Commit message: remove caster physics

File: src/smart_robot/urdf/smart_robot.urdf.xacro (robot description, xacro)
@@ -112,14 +112,9 @@
     </joint>
     <link name="caster_wheel_front_link">
-        <visual><geometry><sphere radius="${wheel_radius*0.5}"/></geometry><material name="grey"><color rgba="0.5 0.5 0.5 1.0"/></material></visual>
-        <collision><geometry><sphere radius="${wheel_radius*0.5}"/></geometry></collision>
+        <visual>
+            <geometry><sphere radius="${wheel_radius*0.5}"/></geometry>
+            <material name="grey"><color rgba="0.5 0.5 0.5 1.0"/></material>
+        </visual>
         <inertial><mass value="${caster_mass}"/><xacro:sphere_inertia m="${caster_mass}" r="${wheel_radius*0.5}"/></inertial>
-        <gazebo reference="caster_wheel_front_link">
-            <mu1>0.05</mu1>
-            <mu2>0.05</mu2>
-            <kp>1000000.0</kp>
-            <kd>100.0</kd>
-            <material>Gazebo/Grey</material>
-        </gazebo>
     </link>
     <joint name="caster_wheel_rear_joint" type="fixed">
@@ -130,5 +125,4 @@
     <link name="caster_wheel_rear_link">
         <visual><geometry><sphere radius="${wheel_radius*0.5}"/></geometry><material name="grey"/></visual>
-        <collision><geometry><sphere radius="${wheel_radius*0.5}"/></geometry></collision>
         <inertial><mass value="${caster_mass}"/><xacro:sphere_inertia m="${caster_mass}" r="${wheel_radius*0.5}"/></inertial>
     </link>

Commit message: fix robot

File: src/smart_robot/urdf/smart_robot.urdf.xacro (robot description, xacro)
@@ -25,5 +25,5 @@
         <parent link="base_footprint"/>
         <child link="base_link"/>
-        <origin xyz="0 0 ${wheel_radius}" rpy="0 0 0"/>
+        <origin xyz="0 0 ${wheel_radius + 0.01 + chassis_height/2}" rpy="0 0 0"/>
     </joint>
     <link name="base_link">
@@ -47,5 +47,5 @@
         <parent link="base_link"/>
         <child link="right_wheel_link"/>
-        <origin xyz="0 -${wheel_separation/2} 0" rpy="0 0 0"/>
+        <origin xyz="0 -${wheel_separation/2} -${0.01 + chassis_height/2}" rpy="0 0 0"/>
         <axis xyz="0 1 0"/>
         <dynamics damping="0.1"/>
@@ -78,5 +78,5 @@
         <parent link="base_link"/>
         <child link="left_wheel_link"/>
-        <origin xyz="0 ${wheel_separation/2} 0" rpy="0 0 0"/>
+        <origin xyz="0 ${wheel_separation/2} -${0.01 + chassis_height/2}" rpy="0 0 0"/>
         <axis xyz="0 1 0"/>
         <dynamics damping="0.1"/>
@@ -109,21 +109,26 @@
         <parent link="base_link"/>
         <child link="caster_wheel_front_link"/>
-        <origin xyz="${chassis_radius*0.8} 0 -${wheel_radius*0.5}" rpy="0 0 0"/>
+        <origin xyz="${chassis_radius*0.8} 0 -${wheel_radius + 0.01 + chassis_height/2 - caster_radius}" rpy="0 0 0"/>
     </joint>
     <link name="caster_wheel_front_link">
-        <visual>
-            <geometry><sphere radius="${wheel_radius*0.5}"/></geometry>
-            <material name="grey"><color rgba="0.5 0.5 0.5 1.0"/></material>
-        </visual>
-        <inertial><mass value="${caster_mass}"/><xacro:sphere_inertia m="${caster_mass}" r="${wheel_radius*0.5}"/></inertial>
+        <visual><geometry><sphere radius="${caster_radius}"/></geometry><material name="grey"><color rgba="0.5 0.5 0.5 1.0"/></material></visual>
+        <collision><geometry><sphere radius="${caster_radius}"/></geometry></collision>
+        <inertial><mass value="${caster_mass}"/><xacro:sphere_inertia m="${caster_mass}" r="${caster_radius}"/></inertial>
+        <gazebo reference="caster_wheel_front_link">
+            <mu1>0.05</mu1> <mu2>0.05</mu2> <material>Gazebo/Grey</material>
+        </gazebo>
     </link>
     <joint name="caster_wheel_rear_joint" type="fixed">
         <parent link="base_link"/>
         <child link="caster_wheel_rear_link"/>
-        <origin xyz="-${chassis_radius*0.8} 0 -${wheel_radius*0.5}" rpy="0 0 0"/>
+        <origin xyz="-${chassis_radius*0.8} 0 -${wheel_radius + 0.01 + chassis_height/2 - caster_radius}" rpy="0 0 0"/>
     </joint>
     <link name="caster_wheel_rear_link">
-        <visual><geometry><sphere radius="${wheel_radius*0.5}"/></geometry><material name="grey"/></visual>
-        <inertial><mass value="${caster_mass}"/><xacro:sphere_inertia m="${caster_mass}" r="${wheel_radius*0.5}"/></inertial>
+        <visual><geometry><sphere radius="${caster_radius}"/></geometry><material name="grey"/></visual>
+        <collision><geometry><sphere radius="${caster_radius}"/></geometry></collision>
+        <inertial><mass value="${caster_mass}"/><xacro:sphere_inertia m="${caster_mass}" r="${caster_radius}"/></inertial>
+        <gazebo reference="caster_wheel_rear_link">
+            <mu1>0.05</mu1> <mu2>0.05</mu2> <material>Gazebo/Grey</material>
+        </gazebo>
     </link>
     <!-- Laser Scanner -->
