Commit message: refine robot

File: src/smart_robot/urdf/smart_robot.urdf.xacro (robot description, xacro)
@@ -42,6 +42,6 @@
         </collision>
         <inertial>
-            <mass value="5.0"/>
-            <xacro:cylinder_inertia m="5.0" r="0.2" h="0.6"/>
+            <mass value="10.0"/>
+            <xacro:cylinder_inertia m="10.0" r="0.2" h="0.6"/>
         </inertial>
     </link>
@@ -123,5 +123,5 @@
         <parent link="right_base"/>
         <child link="right_front_wheel"/>
-        <origin rpy="0 0 0" xyz="0.133333 0 -0.085"/>
+        <origin rpy="0 0 0" xyz="0.18 0 -0.085"/>
         <axis xyz="0 1 0"/>
     </joint>
@@ -144,5 +144,5 @@
         <parent link="right_base"/>
         <child link="right_back_wheel"/>
-        <origin rpy="0 0 0" xyz="-0.133333 0 -0.085"/>
+        <origin rpy="0 0 0" xyz="-0.18 0 -0.085"/>
         <axis xyz="0 1 0"/>
     </joint>
@@ -165,5 +165,10 @@
         <inertial><mass value="0.2"/><xacro:cylinder_inertia m="0.2" r="0.035" h="0.1"/></inertial>
     </link>
-    <joint name="left_front_wheel_joint" type="continuous"><parent link="left_base"/><child link="left_front_wheel"/><origin rpy="0 0 0" xyz="0.133333 0 -0.085"/><axis xyz="0 1 0"/></joint>
+    <joint name="left_front_wheel_joint" type="continuous">
+        <parent link="left_base"/>
+        <child link="left_front_wheel"/>
+        <origin rpy="0 0 0" xyz="0.18 0 -0.085"/>
+        <axis xyz="0 1 0"/>
+    </joint>
     <link name="left_back_wheel">
         <visual><origin rpy="1.57075 0 0" xyz="0 0 0"/><geometry><cylinder length="0.1" radius="0.035"/></geometry><material name="black"/></visual>
@@ -171,5 +176,10 @@
         <inertial><mass value="0.2"/><xacro:cylinder_inertia m="0.2" r="0.035" h="0.1"/></inertial>
     </link>
-    <joint name="left_back_wheel_joint" type="continuous"><parent link="left_base"/><child link="left_back_wheel"/><origin rpy="0 0 0" xyz="-0.133333 0 -0.085"/><axis xyz="0 1 0"/></joint>
+    <joint name="left_back_wheel_joint" type="continuous">
+        <parent link="left_base"/>
+        <child link="left_back_wheel"/>
+        <origin rpy="0 0 0" xyz="-0.18 0 -0.085"/>
+        <axis xyz="0 1 0"/>
+    </joint>
     <link name="sprayer_pole">
         <visual>

Commit message: fix robot

File: src/smart_robot/urdf/smart_robot.urdf.xacro (robot description, xacro)
@@ -3,13 +3,8 @@
     <!-- ================== CONSTANTS & MACROS ================== -->
     <xacro:property name="PI" value="3.1415926535897931"/>
-    <xacro:macro name="box_inertia" params="m x y z">
-        <inertia ixx="${m*(y*y+z*z)/12}" ixy="0" ixz="0" iyy="${m*(x*x+z*z)/12}" iyz="0" izz="${m*(x*x+y*y)/12}"/>
-    </xacro:macro>
-    <xacro:macro name="cylinder_inertia" params="m r h">
-        <inertia ixx="${m*(3*r*r+h*h)/12}" ixy="0" ixz="0" iyy="${m*(3*r*r+h*h)/12}" iyz="0" izz="${m*r*r/2}"/>
-    </xacro:macro>
-    <xacro:macro name="sphere_inertia" params="m r">
-        <inertia ixx="${2*m*r*r/5}" ixy="0" ixz="0" iyy="${2*m*r*r/5}" iyz="0" izz="${2*m*r*r/5}"/>
-    </xacro:macro>
+    <xacro:macro name="box_inertia" params="m x y z"><inertia ixx="${m*(y*y+z*z)/12}" ixy="0" ixz="0" iyy="${m*(x*x+z*z)/12}" iyz="0" izz="${m*(x*x+y*y)/12}"/></xacro:macro>
+    <xacro:macro name="cylinder_inertia" params="m r h"><inertia ixx="${m*(3*r*r+h*h)/12}" ixy="0" ixz="0" iyy="${m*(3*r*r+h*h)/12}" iyz="0" izz="${m*r*r/2}"/></xacro:macro>
+    <xacro:macro name="sphere_inertia" params="m r"><inertia ixx="${2*m*r*r/5}" ixy="0" ixz="0" iyy="${2*m*r*r/5}" iyz="0" izz="${2*m*r*r/5}"/></xacro:macro>
+    <xacro:macro name="wheel_inertia" params="m r h"><inertia ixx="${m*(3*r*r+h*h)/12}" ixy="0" ixz="0" iyy="${m*r*r/2}" iyz="0" izz="${m*(3*r*r+h*h)/12}"/></xacro:macro>
     <!-- ================== MATERIALS ================== -->
     <material name="blue">
@@ -106,45 +101,15 @@
     </joint>
     <link name="right_front_wheel">
-        <visual>
-            <origin rpy="1.57075 0 0" xyz="0 0 0"/>
-            <geometry><cylinder length="0.1" radius="0.035"/></geometry>
-            <material name="black"/>
-        </visual>
-        <collision>
-            <origin rpy="1.57075 0 0" xyz="0 0 0"/>
-            <geometry><cylinder length="0.1" radius="0.035"/></geometry>
-        </collision>
-        <inertial>
-            <mass value="0.2"/>
-            <xacro:cylinder_inertia m="0.2" r="0.035" h="0.1"/>
-        </inertial>
-    </link>
-    <joint name="right_front_wheel_joint" type="continuous">
-        <parent link="right_base"/>
-        <child link="right_front_wheel"/>
-        <origin rpy="0 0 0" xyz="0.18 0 -0.085"/>
-        <axis xyz="0 1 0"/>
-    </joint>
+        <visual><origin rpy="1.57075 0 0"/><geometry><cylinder length="0.1" radius="0.035"/></geometry><material name="black"/></visual>
+        <collision><origin rpy="1.57075 0 0"/><geometry><cylinder length="0.1" radius="0.035"/></geometry></collision>
+        <inertial><mass value="0.2"/><xacro:wheel_inertia m="0.2" r="0.035" h="0.1"/></inertial>
+    </link>
+    <joint name="right_front_wheel_joint" type="continuous"><parent link="right_base"/><child link="right_front_wheel"/><origin xyz="0.18 0 -0.085"/><axis xyz="0 1 0"/></joint>
     <link name="right_back_wheel">
-        <visual>
-            <origin rpy="1.57075 0 0" xyz="0 0 0"/>
-            <geometry><cylinder length="0.1" radius="0.035"/></geometry>
-            <material name="black"/>
-        </visual>
-        <collision>
-            <origin rpy="1.57075 0 0" xyz="0 0 0"/>
-            <geometry><cylinder length="0.1" radius="0.035"/></geometry>
-        </collision>
-        <inertial>
-            <mass value="0.2"/>
-            <xacro:cylinder_inertia m="0.2" r="0.035" h="0.1"/>
-        </inertial>
-    </link>
-    <joint name="right_back_wheel_joint" type="continuous">
-        <parent link="right_base"/>
-        <child link="right_back_wheel"/>
-        <origin rpy="0 0 0" xyz="-0.18 0 -0.085"/>
-        <axis xyz="0 1 0"/>
-    </joint>
+        <visual><origin rpy="1.57075 0 0"/><geometry><cylinder length="0.1" radius="0.035"/></geometry><material name="black"/></visual>
+        <collision><origin rpy="1.57075 0 0"/><geometry><cylinder length="0.1" radius="0.035"/></geometry></collision>
+        <inertial><mass value="0.2"/><xacro:wheel_inertia m="0.2" r="0.035" h="0.1"/></inertial>
+    </link>
+    <joint name="right_back_wheel_joint" type="continuous"><parent link="right_base"/><child link="right_back_wheel"/><origin xyz="-0.18 0 -0.085"/><axis xyz="0 1 0"/></joint>
     <!-- Left Side -->
     <link name="left_leg">
@@ -161,25 +126,15 @@
     <joint name="left_base_joint" type="fixed"><parent link="left_leg"/><child link="left_base"/><origin xyz="0 0 -0.6"/></joint>
     <link name="left_front_wheel">
-        <visual><origin rpy="1.57075 0 0" xyz="0 0 0"/><geometry><cylinder length="0.1" radius="0.035"/></geometry><material name="black"/></visual>
-        <collision><origin rpy="1.57075 0 0" xyz="0 0 0"/><geometry><cylinder length="0.1" radius="0.035"/></geometry></collision>
-        <inertial><mass value="0.2"/><xacro:cylinder_inertia m="0.2" r="0.035" h="0.1"/></inertial>
-    </link>
-    <joint name="left_front_wheel_joint" type="continuous">
-        <parent link="left_base"/>
-        <child link="left_front_wheel"/>
-        <origin rpy="0 0 0" xyz="0.18 0 -0.085"/>
-        <axis xyz="0 1 0"/>
-    </joint>
+        <visual><origin rpy="1.57075 0 0"/><geometry><cylinder length="0.1" radius="0.035"/></geometry><material name="black"/></visual>
+        <collision><origin rpy="1.57075 0 0"/><geometry><cylinder length="0.1" radius="0.035"/></geometry></collision>
+        <inertial><mass value="0.2"/><xacro:wheel_inertia m="0.2" r="0.035" h="0.1"/></inertial>
+    </link>
+    <joint name="left_front_wheel_joint" type="continuous"><parent link="left_base"/><child link="left_front_wheel"/><origin xyz="0.18 0 -0.085"/><axis xyz="0 1 0"/></joint>
     <link name="left_back_wheel">
-        <visual><origin rpy="1.57075 0 0" xyz="0 0 0"/><geometry><cylinder length="0.1" radius="0.035"/></geometry><material name="black"/></visual>
-        <collision><origin rpy="1.57075 0 0" xyz="0 0 0"/><geometry><cylinder length="0.1" radius="0.035"/></geometry></collision>
-        <inertial><mass value="0.2"/><xacro:cylinder_inertia m="0.2" r="0.035" h="0.1"/></inertial>
-    </link>
-    <joint name="left_back_wheel_joint" type="continuous">
-        <parent link="left_base"/>
-        <child link="left_back_wheel"/>
-        <origin rpy="0 0 0" xyz="-0.18 0 -0.085"/>
-        <axis xyz="0 1 0"/>
-    </joint>
+        <visual><origin rpy="1.57075 0 0"/><geometry><cylinder length="0.1" radius="0.035"/></geometry><material name="black"/></visual>
+        <collision><origin rpy="1.57075 0 0"/><geometry><cylinder length="0.1" radius="0.035"/></geometry></collision>
+        <inertial><mass value="0.2"/><xacro:wheel_inertia m="0.2" r="0.035" h="0.1"/></inertial>
+    </link>
+    <joint name="left_back_wheel_joint" type="continuous"><parent link="left_base"/><child link="left_back_wheel"/><origin xyz="-0.18 0 -0.085"/><axis xyz="0 1 0"/></joint>
     <link name="sprayer_pole">
         <visual>
@@ -230,7 +185,7 @@
             <rightJoint>right_front_wheel_joint</rightJoint>
             <rightJoint>right_back_wheel_joint</rightJoint>
-            <wheelSeparation>${2 * 0.22}</wheelSeparation> <!-- 左右腿的距離 -->
+            <wheelSeparation>${2 * 0.22}</wheelSeparation>
             <wheelDiameter>${2 * 0.035}</wheelDiameter>
-            <torque>20</torque>
+            <torque>30</torque>
             <commandTopic>cmd_vel</commandTopic>
             <odometryTopic>odom</odometryTopic>
@@ -238,5 +193,8 @@
             <robotBaseFrame>base_footprint</robotBaseFrame>
             <publishOdomTF>true</publishOdomTF>
+            <publishWheelTF>false</publishWheelTF>
+            <publishWheelJointState>true</publishWheelJointState>
             <odometrySource>world</odometrySource>
+            <legacyMode>false</legacyMode>
         </plugin>
     </gazebo>
@@ -250,14 +208,16 @@
                 <scan>
                     <horizontal>
-                        <samples>90</samples>
+                        <samples>360</samples>
                         <resolution>1</resolution>
-                        <min_angle>-0.785398</min_angle>
-                        <max_angle>0.785398</max_angle>
+                        <min_angle>-3.14</min_angle>
+                        <max_angle>3.14</max_angle>
                     </horizontal>
                 </scan>
-                <range><min>0.10</min><max>10.0</max><resolution>0.01</resolution></range>
-                <noise><type>gaussian</type><mean>0.0</mean><stddev>0.01</stddev></noise>
+                <range>
+                    <min>0.10</min>
+                    <max>10.0</max>
+                </range>
             </ray>
-            <plugin name="gazebo_ros_head_hokuyo_controller" filename="libgazebo_ros_laser.so">
+            <plugin name="gazebo_ros_laser" filename="libgazebo_ros_laser.so">
                 <topicName>/scan</topicName>
                 <frameName>laser_link</frameName>

Commit message: increase tolerance & modify robot laser

File: src/smart_robot/urdf/smart_robot.urdf.xacro (robot description, xacro)
@@ -172,5 +172,5 @@
         <parent link="base_link"/>
         <child link="laser_link"/>
-        <origin xyz="0.2 0 0"/>
+        <origin xyz="0.2 0 -0.15"/>
     </joint>
     <!-- ================== GAZEBO PLUGINS ================== -->
